Commit message: Update codebase: Align axes, add RL drawing node, diagrams, and trained models

File: ros2_ws/src/robot_arm2/urdf/New.xacro (robot description, xacro)
@@ -2,5 +2,5 @@
 <robot name="new" xmlns:xacro="http://www.ros.org/wiki/xacro">
 <xacro:include filename="$(find robot_arm2)/urdf/materials.xacro" />
-<xacro:include filename="$(find robot_arm2)/urdf/new.trans" />
+<xacro:include filename="$(find robot_arm2)/urdf/New.trans" />
 <xacro:include filename="$(find robot_arm2)/urdf/robot_arm2.ros2_control.xacro" />
 <xacro:include filename="$(find robot_arm2)/urdf/robot_arm2.gazebo.xacro" />
@@ -199,5 +199,5 @@
   <parent link="Link4_1"/>
   <child link="Link5_1"/>
-  <axis xyz="1.0 0.0 0.0"/>
+  <axis xyz="-1.0 0.0 0.0"/>
   <limit effort="100" velocity="100"/>
 </joint>
@@ -213,5 +213,5 @@
   <parent link="Link2_1"/>
   <child link="Link3_1"/>
-  <axis xyz="1.0 0.0 0.0"/>
+  <axis xyz="-1.0 0.0 0.0"/>
   <limit effort="100" velocity="100"/>
 </joint>
