Commit message: Remove robot_arm2, rewrite README for visual_servoing
- Delete robot_arm2 package (no longer used)
- Rewrite README: architecture, coordinate frames, training modes
- Fix fk_batch_torch to match exact FK chain from URDF
- Update workspace bounds for base_link -X workspace
- Fix target spawning radius to match 12x12cm ArUco board
- Add reaching target sphere in gazebo visualizer
- Suppress TF_OLD_DATA spam in launch file
- Stabilize drawing pen line with TF grace period

File: ros2_ws/src/visual_servoing/urdf/new_arm/new_arm.xacro (robot description, xacro)
@@ -4,8 +4,9 @@
 <xacro:include filename="$(find visual_servoing)/urdf/new_arm/new_arm.ros2_control.xacro" />
 <xacro:include filename="$(find visual_servoing)/urdf/new_arm/new_arm.gazebo.xacro" />
-<!-- World anchor: 180° yaw so robot arm faces world +X -->
+<!-- World anchor: 180° yaw so robot arm faces world +X
+     Z=-0.209 so end-effector hovers ~5cm above ground at home pose -->
 <link name="world"/>
 <joint name="world_fixed" type="fixed">
-  <origin xyz="0 0 0" rpy="0 0 3.14159265359"/>
+  <origin xyz="0 0 -0.209" rpy="0 0 3.14159265359"/>
   <parent link="world"/>
   <child link="base_link"/>
@@ -857,7 +858,10 @@
   </visual>
 </link>
-<!-- Camera points to world +X, so local yaw=3.14159 -->
+<!-- Camera: mounted above base_link, pitched down to see ArUco board.
+     base_link is at world Z=-0.209, so camera local z=0.85 → world Z≈0.64.
+     Board is at world (0.5, 0, 0.35). Camera yaw=π cancels parent yaw.
+     Pitch=0.57 tilts camera down toward the board. -->
 <joint name="camera_joint" type="fixed">
-  <origin xyz="-0.1 0 0.1" rpy="0 0.6 3.14159265359"/>
+  <origin xyz="-0.05 0 0.85" rpy="0 0.57 3.14159265359"/>
   <parent link="base_link"/>
   <child link="camera_link"/>
