Commit message: feat: gray robot, reduced ArUco log spam, EE ArUco marker, joint fixes
- Define all URDF materials with gray colors (was black due to undefined materials)
- Reduce ArUco detector logging from every 300 to 3000 frames
- Add ArUco marker (ID 4) on end-effector for camera-based EE detection
- Set all joint limits to ±90° (joint 2: -60° to +90°)
- Unify pitch joint axes (2/3/5/6) to +Y direction
- Rewrite gazebo.xacro with correct link names, self_collide=false, gravity=false
- Update README with EE ArUco marker adjustment guide

File: ros2_ws/src/visual_servoing/urdf/new_arm/materials.xacro (robot description, xacro)
@@ -1,6 +1,31 @@
 <?xml version="1.0" ?>
 <robot name="new_arm" xmlns:xacro="http://www.ros.org/wiki/xacro" >
+<!-- Gray tones for robot body (visible in Gazebo Fortress) -->
 <material name="silver">
   <color rgba="0.700 0.700 0.700 1.000"/>
 </material>
+<material name="nylon_66_white">
+  <color rgba="0.750 0.750 0.750 1.000"/>
+</material>
+<material name="steel_satin">
+  <color rgba="0.600 0.600 0.620 1.000"/>
+</material>
+<material name="stainless_steel_satin">
+  <color rgba="0.650 0.650 0.670 1.000"/>
+</material>
+<material name="fabric_white">
+  <color rgba="0.800 0.800 0.800 1.000"/>
+</material>
+<material name="polystyrene">
+  <color rgba="0.700 0.700 0.720 1.000"/>
+</material>
+<material name="opaque212121">
+  <color rgba="0.500 0.500 0.500 1.000"/>
+</material>
+<material name="opaque202209238">
+  <color rgba="0.550 0.550 0.550 1.000"/>
+</material>
+<material name="surface_matte">
+  <color rgba="0.600 0.600 0.600 1.000"/>
+</material>
 </robot>

File: ros2_ws/src/visual_servoing/urdf/new_arm/new_arm.gazebo.xacro (robot description, xacro)
@@ -1,236 +1,70 @@
 <?xml version="1.0" ?>
+<!-- Gazebo Fortress properties for the 6-DOF robot arm.
+     gravity=false:      robot hangs inverted, joints can't fight gravity
+     self_collide=false:  prevents collision-mesh jamming between links -->
 <robot name="new_arm" xmlns:xacro="http://www.ros.org/wiki/xacro" >
-<xacro:property name="body_color" value="Gazebo/Silver" />
-<gazebo reference="base_link">
-  <material>${body_color}</material>
-  <mu1>0.2</mu1>
-  <mu2>0.2</mu2>
-  <self_collide>true</self_collide>
+<!-- Xacro macro to keep things DRY: every link gets no-gravity + no-self-collide -->
+<xacro:macro name="link_gazebo" params="link_name">
+  <gazebo reference="${link_name}">
+    <self_collide>false</self_collide>
+    <gravity>false</gravity>
+    <mu1>0.2</mu1>
+    <mu2>0.2</mu2>
+  </gazebo>
+</xacro:macro>
+<!-- Base & platform -->
+<xacro:link_gazebo link_name="base_link"/>
+<xacro:link_gazebo link_name="old_component__1__1"/>
+<xacro:link_gazebo link_name="old_component__2__1"/>
+<xacro:link_gazebo link_name="old_component__3__1"/>
+<xacro:link_gazebo link_name="old_component__4__1"/>
+<xacro:link_gazebo link_name="old_component__5__1"/>
+<xacro:link_gazebo link_name="old_component__6__1"/>
+<xacro:link_gazebo link_name="old_component__7__1"/>
+<xacro:link_gazebo link_name="old_component__8__1"/>
+<xacro:link_gazebo link_name="old_component__9__1"/>
+<xacro:link_gazebo link_name="old_component__10__1"/>
+<xacro:link_gazebo link_name="old_component__11__1"/>
+<xacro:link_gazebo link_name="old_component__12__1"/>
+<xacro:link_gazebo link_name="old_component__13__1"/>
+<!-- Servo mounts & arm links -->
+<xacro:link_gazebo link_name="old_component__14__1"/>
+<xacro:link_gazebo link_name="old_component__15__1"/>
+<xacro:link_gazebo link_name="old_component__16__1"/>
+<xacro:link_gazebo link_name="old_component__17__1"/>
+<xacro:link_gazebo link_name="old_component__18__1"/>
+<xacro:link_gazebo link_name="old_component__19__1"/>
+<xacro:link_gazebo link_name="old_component__20__1"/>
+<xacro:link_gazebo link_name="old_component__21__1"/>
+<xacro:link_gazebo link_name="old_component__22__1"/>
+<xacro:link_gazebo link_name="old_component__23__1"/>
+<xacro:link_gazebo link_name="old_component__24__1"/>
+<xacro:link_gazebo link_name="old_component__25__1"/>
+<!-- Pen / end-effector -->
+<xacro:link_gazebo link_name="giabut_1"/>
+<xacro:link_gazebo link_name="but_1"/>
+<xacro:link_gazebo link_name="bibut_1"/>
+<!-- Base bolts -->
+<xacro:link_gazebo link_name="old_component__29__1"/>
+<xacro:link_gazebo link_name="old_component__30__1"/>
+<xacro:link_gazebo link_name="old_component__31__1"/>
+<xacro:link_gazebo link_name="old_component__32__1"/>
+<!-- End-effector ArUco marker -->
+<gazebo reference="ee_aruco_marker">
+  <self_collide>false</self_collide>
   <gravity>false</gravity>
+  <visual>
+    <material>
+      <diffuse>1 1 1 1</diffuse>
+      <specular>0.1 0.1 0.1 1</specular>
+      <pbr>
+        <metal>
+          <albedo_map>model://aruco_marker_4/materials/textures/marker_4.png</albedo_map>
+        </metal>
+      </pbr>
+    </material>
+  </visual>
 </gazebo>
-<gazebo reference="canh1_1">
-  <material>${body_color}</material>
-  <mu1>0.2</mu1>
-  <mu2>0.2</mu2>
-  <self_collide>true</self_collide>
-  <gravity>false</gravity>
-</gazebo>
-<gazebo reference="canh2_1">
-  <material>${body_color}</material>
-  <mu1>0.2</mu1>
-  <mu2>0.2</mu2>
-  <self_collide>true</self_collide>
-  <gravity>false</gravity>
-</gazebo>
-<gazebo reference="canh3_1">
-  <material>${body_color}</material>
-  <mu1>0.2</mu1>
-  <mu2>0.2</mu2>
-  <self_collide>true</self_collide>
-  <gravity>false</gravity>
-</gazebo>
-<gazebo reference="canh4_1">
-  <material>${body_color}</material>
-  <mu1>0.2</mu1>
-  <mu2>0.2</mu2>
-  <self_collide>true</self_collide>
-  <gravity>false</gravity>
-</gazebo>
-<gazebo reference="gia1_1">
-  <material>${body_color}</material>
-  <mu1>0.2</mu1>
-  <mu2>0.2</mu2>
-  <self_collide>true</self_collide>
-  <gravity>false</gravity>
-</gazebo>
-<gazebo reference="gia2_1">
-  <material>${body_color}</material>
-  <mu1>0.2</mu1>
-  <mu2>0.2</mu2>
-  <self_collide>true</self_collide>
-  <gravity>false</gravity>
-</gazebo>
-<gazebo reference="basetren_1">
-  <material>${body_color}</material>
-  <mu1>0.2</mu1>
-  <mu2>0.2</mu2>
-  <self_collide>true</self_collide>
-  <gravity>false</gravity>
-</gazebo>
-<gazebo reference="dongco1_1">
-  <material>${body_color}</material>
-  <mu1>0.2</mu1>
-  <mu2>0.2</mu2>
-  <self_collide>true</self_collide>
-  <gravity>false</gravity>
-</gazebo>
-<gazebo reference="dongco2_1">
-  <material>${body_color}</material>
-  <mu1>0.2</mu1>
-  <mu2>0.2</mu2>
-  <self_collide>true</self_collide>
-  <gravity>false</gravity>
-</gazebo>
-<gazebo reference="dongco3_1">
-  <material>${body_color}</material>
-  <mu1>0.2</mu1>
-  <mu2>0.2</mu2>
-  <self_collide>true</self_collide>
-  <gravity>false</gravity>
-</gazebo>
-<gazebo reference="dongco4_1">
-  <material>${body_color}</material>
-  <mu1>0.2</mu1>
-  <mu2>0.2</mu2>
-  <self_collide>true</self_collide>
-  <gravity>false</gravity>
-</gazebo>
-<gazebo reference="quat1_1">
-  <material>${body_color}</material>
-  <mu1>0.2</mu1>
-  <mu2>0.2</mu2>
-  <self_collide>true</self_collide>
-  <gravity>false</gravity>
-</gazebo>
-<gazebo reference="quat2_1">
-  <material>${body_color}</material>
-  <mu1>0.2</mu1>
-  <mu2>0.2</mu2>
-  <self_collide>true</self_collide>
-  <gravity>false</gravity>
-</gazebo>
-<gazebo reference="quat3_1">
-  <material>${body_color}</material>
-  <mu1>0.2</mu1>
-  <mu2>0.2</mu2>
-  <self_collide>true</self_collide>
-  <gravity>false</gravity>
-</gazebo>
-<gazebo reference="quat4_1">
-  <material>${body_color}</material>
-  <mu1>0.2</mu1>
-  <mu2>0.2</mu2>
-  <self_collide>true</self_collide>
-  <gravity>false</gravity>
-</gazebo>
-<gazebo reference="pinpi_1">
-  <material>${body_color}</material>
-  <mu1>0.2</mu1>
-  <mu2>0.2</mu2>
-  <self_collide>true</self_collide>
-  <gravity>false</gravity>
-</gazebo>
-<gazebo reference="hopdo_1">
-  <material>${body_color}</material>
-  <mu1>0.2</mu1>
-  <mu2>0.2</mu2>
-  <self_collide>true</self_collide>
-  <gravity>false</gravity>
-</gazebo>
-<gazebo reference="basearm_1">
-  <material>${body_color}</material>
-  <mu1>0.2</mu1>
-  <mu2>0.2</mu2>
-  <self_collide>true</self_collide>
-  <gravity>false</gravity>
-</gazebo>
-<gazebo reference="sv1_1">
-  <material>${body_color}</material>
-  <mu1>0.2</mu1>
-  <mu2>0.2</mu2>
-  <self_collide>true</self_collide>
-  <gravity>false</gravity>
-</gazebo>
-<gazebo reference="link1_1">
-  <material>${body_color}</material>
-  <mu1>0.2</mu1>
-  <mu2>0.2</mu2>
-  <self_collide>true</self_collide>
-  <gravity>false</gravity>
-</gazebo>
-<gazebo reference="sv2_1">
-  <material>${body_color}</material>
-  <mu1>0.2</mu1>
-  <mu2>0.2</mu2>
-  <self_collide>true</self_collide>
-  <gravity>false</gravity>
-</gazebo>
-<gazebo reference="link2_1">
-  <material>${body_color}</material>
-  <mu1>0.2</mu1>
-  <mu2>0.2</mu2>
-  <self_collide>true</self_collide>
-  <gravity>false</gravity>
-</gazebo>
-<gazebo reference="sv3_1">
-  <material>${body_color}</material>
-  <mu1>0.2</mu1>
-  <mu2>0.2</mu2>
-  <self_collide>true</self_collide>
-  <gravity>false</gravity>
-</gazebo>
-<gazebo reference="link3_1">
-  <material>${body_color}</material>
-  <mu1>0.2</mu1>
-  <mu2>0.2</mu2>
-  <self_collide>true</self_collide>
-  <gravity>false</gravity>
-</gazebo>
-<gazebo reference="sv4_1">
-  <material>${body_color}</material>
-  <mu1>0.2</mu1>
-  <mu2>0.2</mu2>
-  <self_collide>true</self_collide>
-  <gravity>false</gravity>
-</gazebo>
-<gazebo reference="link4_1">
-  <material>${body_color}</material>
-  <mu1>0.2</mu1>
-  <mu2>0.2</mu2>
-  <self_collide>true</self_collide>
-  <gravity>false</gravity>
-</gazebo>
-<gazebo reference="sv5_1">
-  <material>${body_color}</material>
-  <mu1>0.2</mu1>
-  <mu2>0.2</mu2>
-  <self_collide>true</self_collide>
-  <gravity>false</gravity>
-</gazebo>
-<gazebo reference="link5_1">
-  <material>${body_color}</material>
-  <mu1>0.2</mu1>
-  <mu2>0.2</mu2>
-  <self_collide>true</self_collide>
-  <gravity>false</gravity>
-</gazebo>
-<gazebo reference="sv6_1">
-  <material>${body_color}</material>
-  <mu1>0.2</mu1>
-  <mu2>0.2</mu2>
-  <self_collide>true</self_collide>
-  <gravity>false</gravity>
-</gazebo>
-<gazebo reference="giabut_1">
-  <material>${body_color}</material>
-  <mu1>0.2</mu1>
-  <mu2>0.2</mu2>
-  <self_collide>true</self_collide>
-  <gravity>false</gravity>
-</gazebo>
-<gazebo reference="but_1">
-  <material>${body_color}</material>
-  <mu1>0.2</mu1>
-  <mu2>0.2</mu2>
-  <self_collide>true</self_collide>
-  <gravity>false</gravity>
-</gazebo>
-<gazebo reference="bibut_1">
-  <material>${body_color}</material>
-  <mu1>0.2</mu1>
-  <mu2>0.2</mu2>
-  <self_collide>true</self_collide>
-  <gravity>false</gravity>
-</gazebo>
+<!-- ========== CAMERA SENSOR ========== -->
 <gazebo reference="camera_link">
   <sensor name="camera" type="camera">

File: ros2_ws/src/visual_servoing/urdf/new_arm/new_arm.xacro (robot description, xacro)
@@ -752,5 +752,5 @@
   <child link="old_component__16__1"/>
   <axis xyz="0.0 0.0 -1.0"/>
-  <limit upper="3.141593" lower="-3.141593" effort="100" velocity="100"/>
+  <limit upper="1.5708" lower="-1.5708" effort="100" velocity="100"/>
 </joint>
 <joint name="Rigid 21" type="fixed">
@@ -763,6 +763,6 @@
   <parent link="old_component__17__1"/>
   <child link="old_component__18__1"/>
-  <axis xyz="-0.0 -1.0 -0.0"/>
-  <limit upper="1.570796" lower="-1.570796" effort="100" velocity="100"/>
+  <axis xyz="0.0 1.0 0.0"/>
+  <limit upper="1.5708" lower="-1.0472" effort="100" velocity="100"/>
 </joint>
 <joint name="Revolute 23" type="revolute">
@@ -770,6 +770,6 @@
   <parent link="old_component__18__1"/>
   <child link="old_component__19__1"/>
-  <axis xyz="0.0 -1.0 -0.0"/>
-  <limit upper="3.141593" lower="-0.785398" effort="100" velocity="100"/>
+  <axis xyz="0.0 1.0 0.0"/>
+  <limit upper="1.5708" lower="-1.5708" effort="100" velocity="100"/>
 </joint>
 <joint name="Rigid 24" type="fixed">
@@ -788,5 +788,5 @@
   <child link="old_component__22__1"/>
   <axis xyz="0.0 0.0 -1.0"/>
-  <limit upper="3.141593" lower="-3.141593" effort="100" velocity="100"/>
+  <limit upper="1.5708" lower="-1.5708" effort="100" velocity="100"/>
 </joint>
 <joint name="Rigid 27" type="fixed">
@@ -799,6 +799,6 @@
   <parent link="old_component__23__1"/>
   <child link="old_component__24__1"/>
-  <axis xyz="-0.0 -1.0 -0.0"/>
-  <limit upper="2.356194" lower="-2.356194" effort="100" velocity="100"/>
+  <axis xyz="0.0 1.0 0.0"/>
+  <limit upper="1.5708" lower="-1.5708" effort="100" velocity="100"/>
 </joint>
 <joint name="Rigid 29" type="fixed">
@@ -812,5 +812,5 @@
   <child link="giabut_1"/>
   <axis xyz="0.0 1.0 0.0"/>
-  <limit upper="3.141593" lower="0.0" effort="100" velocity="100"/>
+  <limit upper="1.5708" lower="-1.5708" effort="100" velocity="100"/>
 </joint>
 <joint name="Rigid 32" type="fixed">
@@ -823,4 +823,29 @@
   <parent link="but_1"/>
   <child link="bibut_1"/>
+</joint>
+<!-- ========== ARUCO MARKER (ID 4) ON END-EFFECTOR ========== -->
+<!-- Small ArUco marker attached to the pen for camera-based end-effector detection.
+     Positioned to the right of the pen (local +Y), facing outward so the overhead
+     camera can see it. The marker face normal points along local +Y. -->
+<link name="ee_aruco_marker">
+  <inertial>
+    <mass value="0.001"/>
+    <inertia ixx="1e-07" iyy="1e-07" izz="1e-07" ixy="0" iyz="0" ixz="0"/>
+  </inertial>
+  <visual>
+    <origin xyz="0 0 0" rpy="0 0 0"/>
+    <geometry>
+      <box size="0.020 0.001 0.020"/>
+    </geometry>
+    <material name="aruco_white">
+      <color rgba="1.0 1.0 1.0 1.0"/>
+    </material>
+  </visual>
+</link>
+<joint name="ee_aruco_joint" type="fixed">
+  <!-- Offset: 25mm to the right of pen center, 15mm forward, rotated so marker face is visible from above -->
+  <origin xyz="-0.015 0.025 -0.015" rpy="1.5708 0 0"/>
+  <parent link="but_1"/>
+  <child link="ee_aruco_marker"/>
 </joint>
 <joint name="Revolute 34" type="fixed">
