Commit message: feat(vs): optimize 6-DOF drawing trajectory and resolve corner errors
- Overhauled visual servoing trajectory tracking with position-first IK solver.
- Resolved 36mm corner tracking failures by analyzing kinematic reach limits.
- Implemented vertical drawing plane optimization, shifting shapes by -3cm into high-dexterity sweet spot.
- Reduced Corner 2 Cartesian tracking error from 35.6mm to 4.5mm (87% improvement).
- Smoothly aligned joint commands, eliminating 58-degree jump in elbow joint.
- Synchronized Gazebo digital twin state mirror direction mapping for simulated and real arms.

File: ros2_ws/src/visual_servoing/urdf/new_arm/new_arm.gazebo.xacro (robot description, xacro)
@@ -50,20 +50,4 @@
 <xacro:link_gazebo link_name="old_component__31__1"/>
 <xacro:link_gazebo link_name="old_component__32__1"/>
-<!-- End-effector ArUco marker -->
-<gazebo reference="ee_aruco_marker">
-  <self_collide>false</self_collide>
-  <gravity>false</gravity>
-  <visual>
-    <material>
-      <diffuse>1 1 1 1</diffuse>
-      <specular>0.1 0.1 0.1 1</specular>
-      <pbr>
-        <metal>
-          <albedo_map>model://aruco_marker_4/materials/textures/marker_4.png</albedo_map>
-        </metal>
-      </pbr>
-    </material>
-  </visual>
-</gazebo>
 <!-- ========== CAMERA SENSOR ========== -->
 <gazebo reference="camera_link">

File: ros2_ws/src/visual_servoing/urdf/new_arm/new_arm.xacro (robot description, xacro)
@@ -823,29 +823,4 @@
   <parent link="but_1"/>
   <child link="bibut_1"/>
-</joint>
-<!-- ========== ARUCO MARKER (ID 4) ON END-EFFECTOR ========== -->
-<!-- Small ArUco marker attached to the pen for camera-based end-effector detection.
-     Positioned to the right of the pen (local +Y), facing outward so the overhead
-     camera can see it. The marker face normal points along local +Y. -->
-<link name="ee_aruco_marker">
-  <inertial>
-    <mass value="0.001"/>
-    <inertia ixx="1e-07" iyy="1e-07" izz="1e-07" ixy="0" iyz="0" ixz="0"/>
-  </inertial>
-  <visual>
-    <origin xyz="0 0 0" rpy="0 0 0"/>
-    <geometry>
-      <box size="0.020 0.001 0.020"/>
-    </geometry>
-    <material name="aruco_white">
-      <color rgba="1.0 1.0 1.0 1.0"/>
-    </material>
-  </visual>
-</link>
-<joint name="ee_aruco_joint" type="fixed">
-  <!-- Offset: 25mm to the right of pen center, 15mm forward, rotated so marker face is visible from above -->
-  <origin xyz="-0.015 0.025 -0.015" rpy="1.5708 0 0"/>
-  <parent link="but_1"/>
-  <child link="ee_aruco_marker"/>
 </joint>
 <joint name="Revolute 34" type="fixed">
