Commit message: feat: stabilize digital twin pipeline and add PID tuning
- Implemented FastDDS Discovery Server setup in launch config for robust Sim-to-Real Mirroring
- Updated Gazebo GZ_IP to localhost to prevent multicast Pi crashing
- Fixed joint rotation mirroring and trajectory server name mismatches
- Updated ROS 2 Humble setup and network instructions in README
- Finalized PID real-time reinforcement learning pipeline integration

File: ros2_ws/src/visual_servoing/urdf/new_arm/new_arm.ros2_control.xacro (robot description, xacro)
@@ -50,6 +50,6 @@
     <joint name="Revolute 22">
       <command_interface name="position">
-        <param name="min">-1.57</param>
-        <param name="max">1.57</param>
+        <param name="min">-3.14</param>
+        <param name="max">3.14</param>
       </command_interface>
       <state_interface name="position"/>
@@ -82,5 +82,5 @@
     <joint name="Revolute 30">
       <command_interface name="position">
-        <param name="min">0.0</param>
+        <param name="min">-3.14</param>
         <param name="max">3.14</param>
       </command_interface>

File: ros2_ws/src/visual_servoing/urdf/new_arm/new_arm.xacro (robot description, xacro)
@@ -763,5 +763,5 @@
   <parent link="old_component__17__1"/>
   <child link="old_component__18__1"/>
-  <axis xyz="0.0 1.0 0.0"/>
+  <axis xyz="0.0 -1.0 0.0"/>
   <limit upper="1.5708" lower="-1.0472" effort="100" velocity="100"/>
 </joint>
@@ -787,6 +787,6 @@
   <parent link="old_component__21__1"/>
   <child link="old_component__22__1"/>
-  <axis xyz="0.0 0.0 -1.0"/>
-  <limit upper="1.5708" lower="-1.5708" effort="100" velocity="100"/>
+  <axis xyz="0.0 0.0 1.0"/>
+  <limit upper="3.1415" lower="-3.1415" effort="100" velocity="100"/>
 </joint>
 <joint name="Rigid 27" type="fixed">
@@ -799,5 +799,5 @@
   <parent link="old_component__23__1"/>
   <child link="old_component__24__1"/>
-  <axis xyz="0.0 1.0 0.0"/>
+  <axis xyz="0.0 -1.0 0.0"/>
   <limit upper="1.5708" lower="-1.5708" effort="100" velocity="100"/>
 </joint>

Commit message: Enforce Joint 4 lock at 90 deg and sync digital twin state mirror

File: ros2_ws/src/visual_servoing/urdf/new_arm/new_arm.ros2_control.xacro (robot description, xacro)
@@ -66,6 +66,6 @@
     <joint name="Revolute 26">
       <command_interface name="position">
-        <param name="min">-3.14</param>
-        <param name="max">3.14</param>
+        <param name="min">0.0</param>
+        <param name="max">3.14159</param>
       </command_interface>
       <state_interface name="position"/>

File: ros2_ws/src/visual_servoing/urdf/new_arm/new_arm.xacro (robot description, xacro)
@@ -784,9 +784,9 @@
 </joint>
 <joint name="Revolute 26" type="revolute">
-  <origin xyz="0.0 -0.00995 -0.0148" rpy="0 0 0"/>
+  <origin xyz="0.0 -0.00995 -0.0148" rpy="0 0 -1.570796"/>
   <parent link="old_component__21__1"/>
   <child link="old_component__22__1"/>
   <axis xyz="0.0 0.0 1.0"/>
-  <limit upper="3.1415" lower="-3.1415" effort="100" velocity="100"/>
+  <limit upper="1.5708" lower="-1.5708" effort="100" velocity="100"/>
 </joint>
 <joint name="Rigid 27" type="fixed">
